File: ZoumoBotRio.kicad_pcb (KiCad board)
At the start: 2 copper layers, 89.7 x 54.9 mm, 211 parts, among them CON1 BARREL_JACK, J1 Screw_Terminal_1x05, J2 Screw_Terminal_1x05, P1 USB_OTG, P10 A1, P11 D1, P12 A0, P13 D0, P14 CONN_01X06, P2 A5, P3 D7, P4 A4, P5 D6, P6 A3, P7 D5, P8 A2, P9 D4, Q1 Q_PMOS_GDS, Q2 IR Receiver, Q3 IR Receiver, U1 ZLDO1117K50TC, U2 ATmega32U4, U3 SOT361-1_2, U4 TB6612FNG, U5 TB6612FNG, Y1 16MHz

Commit message: Tweaked Back Silkscreen
Other:
- board text added: "Designed by Patrick Smith 2017"
Changed lines of the file:
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@@
     (links 379)
     (no_connects 2)
-    (area 104.064999 84.245949 193.884051 139.274051)
+    (area 76.124999 81.204999 200.735001 139.700001)
     (thickness 1.6)
-    (drawings 39)
+    (drawings 40)
     (tracks 1012)
     (zones 0)
@@
     (34 B.Paste user)
     (35 F.Paste user)
-    (36 B.SilkS user hide)
+    (36 B.SilkS user)
     (37 F.SilkS user)
     (38 B.Mask user)
@@
     (pad_to_mask_clearance 0.2)
     (aux_axis_origin 0 0)
-    (visible_elements 7FFF777F)
+    (visible_elements 7FFFF77F)
     (pcbplotparams
       (layerselection 0x00030_80000001)
@@
       (net 2 GND) (zone_connect 2))
   )
+  (gr_text "Designed by Patrick Smith\n2017" (at 124.333 91.948) (layer B.SilkS)
+    (effects (font (size 1 1) (thickness 0.15) italic) (justify mirror))
+  )
   (gr_line (start 159.385 134.62) (end 161.925 137.16) (layer Edge.Cuts) (width 0.15))
